File: speedy/speedy.sch (KiCad schematic (older format))
At the start: 15 parts

Commit message: projekt1.1
Parts:
- added BT?: Battery_Cell, symbol Battery_Cell
- added BZ?: Buzzer, symbol Buzzer
- added C?: CP1_Small, symbol CP1_Small
- added C? (x2): C, symbol C
- added MCP?: ArduinoMicro, symbol ArduinoMicro
- added Q?: Q_NPN_BCE, symbol Q_NPN_BCE
- added Q?: Q_PMOS_GDS, symbol Q_PMOS_GDS
- added R? (x15): R, symbol R
- added U?: CD74HC4067, symbol CD74HC4067
- added U?: SW1, symbol SW1
- added U?: SN754410, symbol SN754410
- added U? (x2): Motor, symbol Motor
- added U?: RN42, symbol RN42
- added U? (x2): LD1117V33, symbol LD1117V33
Connections:
- net +5V: now also MCP?.29 (+5V), R?.2, R?.2, R?.2, R?.2, R?.2, R?.2, R?.2, R?.2, R?.2, R?.2, R?.2, U?.1 (1,2_EN), U?.24 (VCC), U?.3 (VCC5), U?.3 (VCC5), U?.3 (VIN), U?.9 (3,4_EN)
- net +9V: now also MCP?.32 (VIN), Q?.2 (D), R?.2, U?.16 (VCC2), U?.8 (VCC1)
- net GND: now also BT?.2 (-), BZ?.2 (+), C?.2, MCP?.31 (GND), Q?.3 (E), R?.1, U?.1 (GND), U?.1 (GND), U?.1 (GND), U?.12 (GND), U?.12 (GND), U?.12 (GND), U?.13 (GND), U?.15 (ENABLE), U?.28 (GND), U?.29 (GND), U?.3, U?.4 (GND), U?.5 (GND), U?.6 (GND), U?.6 (GND)
- net LS1: now reaches S?.3 (C3)
- net LS1: now also R?.1, U?.9 (I0)
- net LS2: now reaches S?.3 (C3)
- net LS2: now also R?.1, U?.8 (I1)
- net LS3: now reaches S?.3 (C3)
- net LS3: now also R?.1, U?.7 (I2)
- net LS4: now reaches S?.3 (C3)
- net LS4: now also R?.1, U?.6 (I3)
- net LS5: now reaches S?.3 (C3)
- net LS5: now also R?.1, U?.5 (I4)
- net at S?.2 (L2): now also S?.2 (L2), Q?.2 (C)
- net LS6: now reaches S?.3 (C3)
- net LS6: now also R?.1, U?.4 (I5)
- net LS7: now reaches S?.3 (C3)
- net LS7: now also R?.1, U?.3 (I6)
- net LS8: now reaches S?.3 (C3)
- net LS8: now also R?.1, U?.2 (I7)
- net LS9: now reaches S?.3 (C3)
- net LS9: now also R?.1, U?.23 (I8)
- net LS10: now reaches S?.3 (C3)
- net LS10: now also R?.1, U?.22 (I9)
- net LS11: now reaches S?.3 (C3)
- net LS11: now also R?.1, U?.21 (I10)
- new net: Q?.1 (B), R?.2
- new net: Q?.1 (G), R?.2, U?.2
- new net: C?.2, U?.11 (3Y), U?.2 (M2)
- new net: C?.1, U?.1 (M1), U?.14 (4Y)
- new net: C?.2, U?.2 (M2), U?.6 (2Y)
- new net: C?.1, U?.1 (M1)
- new net: U?.11 (VDD), U?.2 (VOUT)
- new net: U?.13 (UART_RX), U?.2 (VOUT)
- new net +9VA: BT?.1 (+), C?.1, Q?.3 (S), R?.1, U?.1
- new net BUZZ: BZ?.1 (-)
- new net B_RX: U?.3 (VIN)
- new net B_TX: U?.14 (UART_TX)
- new net C0: U?.10 (S0)
- new net C1: U?.11 (S1)
- new net C2: U?.14 (S2)
- new net C3: U?.13 (S3)
- new net CD1: U?.10 (3A)
- new net CD2: U?.15 (4A)
- new net CL1: U?.2 (1A)
- new net CL2: U?.7 (2A)
- new net MD1: U?.4 (OutA)
- new net MD2: U?.5 (OutB)
- new net ML1: U?.4 (OutA)
- new net ML2: U?.5 (OutB)
- new net VBAT: R?.1, R?.2
- no-connect marks 0 -> 37
Other:
- moved on the sheet: D?, R?, S?

Commit message: projekt
spremembe 17.3.2017
Parts:
- removed D?: LED, symbol LED
- removed R?: 1 K, symbol R
- removed R? (x3): R, symbol R
- removed S? (x3): qre1113, symbol qre1113
- removed U? (x2): LD1117V33, symbol LD1117V33
- added R?: 220, symbol R
- added R? (x4): 10K, symbol R
- added S? (x3): qre1113, symbol qre1113
- added U?: TXB0104-Q1, symbol TXB0104-Q1
- added U?: BUT_SW, symbol BUT_SW
- BT?: value Battery_Cell -> Battery_Cell 9V
- C?: value CP1_Small -> 22uF
- R? (x2): value R -> 150
- R? (x11): value R -> 10K
- R?: value R -> 1K
Connections:
- net +5V: now also R?.1, R?.2, R?.2, R?.2, U?.14 (VCCB)
- net +9V: now also R?.1
- net BUZZ: now also MCP?.18 (13(PWM))
- net C0: now also MCP?.24 (A3)
- net C1: now also MCP?.25 (A4)
- net C2: now also MCP?.26 (A5)
- net C3: now also MCP?.9 (4/A6)
- net CL1: now also MCP?.10 (5(PWM))
- net CL2: now also MCP?.11 (6(PWM)/A7)
- net GND: now also MCP?.6 (GND), S?.4 (E4), S?.4 (E4), S?.4 (E4), U?.2, U?.7 (OE)
- net LS10: now also R?.1, S?.3 (C3); no longer R?.1, S?.3 (C3)
- net LS11: now also R?.1, S?.3 (C3)
- net LS5: now also R?.1, S?.3 (C3)
- net LS6: now also R?.1, S?.3 (C3)
- net LS7: now also R?.1, S?.3 (C3); no longer R?.1, S?.3 (C3)
- net LS8: now also R?.1, S?.3 (C3); no longer R?.1, S?.3 (C3)
- net LS9: now also R?.1, S?.3 (C3); no longer R?.1, S?.3 (C3)
- net MD1: now also MCP?.7 (2/SDA)
- net MD2: now also MCP?.8 (3(PWM)/SCL)
- net ML1: now also MCP?.3 (1/TX)
- net ML2: now also MCP?.4 (0/RX)
- net VBAT: now also MCP?.22 (A1)
- net at S?.2 (L2): now also Q?.2 (C), S?.2 (L2)
- net XY: now reaches R?.1
- net XY: now also MCP?.23 (A2)
- net BTX: now reaches MCP?.12 (7)
- net BTX: now also U?.13 (B1)
- net BRX: now reaches MCP?.13 (8/A8)
- net BRX: now also U?.12 (B2)
- net CR1: now reaches MCP?.14 (9(PWM)/A9)
- net CR2: now reaches MCP?.15 (10(PWM)/A10)
- net BUT: now reaches MCP?.16 (11(PWM))
- net BUT: now also R?.2, U?.1
- net +3V3: now reaches MCP?.19 (3.3V)
- net +3V3: now also U?.11 (VDD), U?.1 (VCCA), U?.7 (OE)
- net MUX: now reaches MCP?.21 (A0)
- net MUX: now also U?.1 (COMMON)
- net at U?.3 (1Y): now also C?.1, U?.1 (M1)
- net at U?.13 (UART_RX): now also U?.3 (A2)
- net B_TX: no longer names the net of U?.14 (UART_TX)
- net B_TX: now also U?.2 (A1)
- new net: R?.2, S?.1 (L1)
- new net: S?.1 (L1), S?.2 (L2) (x2)
- no-connect marks 37 -> 45
